Commit message: inertial complete

File: steering_wheel_chassis/urdf/steering_wheel_chassis.urdf (robot description, URDF)
Before this commit: robot steering_wheel_chassis, 13 links, 12 joints
Links:
- link L_B_sW_Link: mass 0.000678584013175396 -> 0.1
- link L_F_sW_Link: mass 0.000678584013175396 -> 0.1
- link R_B_sW_Link: mass 0.000678584013175396 -> 0.1
- link R_F_sW_Link: mass 0.000678584013175396 -> 0.1
