Commit message: r2 up&down completely

File: stee_new/stee_new/urdf/stee_new.urdf (robot description, URDF)
Before this commit: robot stee_new, 15 links, 14 joints
Links:
- link L_B_S_wheel_Link: mass 0.0012284 -> 0.1
- link L_F_S_wheel_Link: mass 0.0012284 -> 0.1
- link R_B_S_wheel_Link: mass 0.0012284 -> 0.1
- link R_F_S_wheel_Link: mass 0.0012284 -> 0.1
- link base_link: mass 9.11525644204073 -> 15.11525644204073

File: steering_wheel_chassis/urdf/steering_wheel__robot.xacro (robot description, xacro)
@@ -13,3 +13,39 @@
         </plugin>
     </gazebo>
+<gazebo reference="L_F_S_wheel_Link">
+        <mu1>0.1</mu1>          <!-- 法向摩擦系数（主） -->
+        <mu2>0.1</mu2>          <!-- 切向摩擦系数（次） -->
+        <!-- <fdir1>0 0 0</fdir1>    摩擦方向（0 0 0 表示各向同性） -->
+        <!-- <slip1>0.01</slip1>     纵向滑移系数（可选：增大=更滑） -->
+        <!-- <slip2>0.01</slip2>     横向滑移系数（可选：增大=更滑） -->
+      <rolling>0.001</rolling>  <!-- 滚动摩擦系数（越小=滚动越顺滑） -->
+      <torque>0.001</torque>    <!-- 旋转摩擦扭矩（越小=旋转阻力越小） -->
+</gazebo>
+<gazebo reference="L_B_S_wheel_Link">
+        <mu1>0.1</mu1>          <!-- 法向摩擦系数（主） -->
+        <mu2>0.1</mu2>          <!-- 切向摩擦系数（次） -->
+        <!-- <fdir1>0 0 0</fdir1>    摩擦方向（0 0 0 表示各向同性） -->
+        <!-- <slip1>0.01</slip1>     纵向滑移系数（可选：增大=更滑） -->
+        <!-- <slip2>0.01</slip2>     横向滑移系数（可选：增大=更滑） -->
+      <rolling>0.001</rolling>  <!-- 滚动摩擦系数（越小=滚动越顺滑） -->
+      <torque>0.001</torque>    <!-- 旋转摩擦扭矩（越小=旋转阻力越小） -->
+</gazebo>
+<gazebo reference="R_F_S_wheel_Link">
+        <mu1>0.1</mu1>          <!-- 法向摩擦系数（主） -->
+        <mu2>0.1</mu2>          <!-- 切向摩擦系数（次） -->
+        <!-- <fdir1>0 0 0</fdir1>    摩擦方向（0 0 0 表示各向同性） -->
+        <!-- <slip1>0.01</slip1>     纵向滑移系数（可选：增大=更滑） -->
+        <!-- <slip2>0.01</slip2>     横向滑移系数（可选：增大=更滑） -->
+      <rolling>0.001</rolling>  <!-- 滚动摩擦系数（越小=滚动越顺滑） -->
+      <torque>0.001</torque>    <!-- 旋转摩擦扭矩（越小=旋转阻力越小） -->
+</gazebo>
+<gazebo reference="R_B_S_wheel_Link">
+        <mu1>0.1</mu1>          <!-- 法向摩擦系数（主） -->
+        <mu2>0.1</mu2>          <!-- 切向摩擦系数（次） -->
+        <!-- <fdir1>0 0 0</fdir1>    摩擦方向（0 0 0 表示各向同性） -->
+        <!-- <slip1>0.01</slip1>     纵向滑移系数（可选：增大=更滑） -->
+        <!-- <slip2>0.01</slip2>     横向滑移系数（可选：增大=更滑） -->
+      <rolling>0.001</rolling>  <!-- 滚动摩擦系数（越小=滚动越顺滑） -->
+      <torque>0.001</torque>    <!-- 旋转摩擦扭矩（越小=旋转阻力越小） -->
+</gazebo>
 </robot>
