Commit message: 3 joint work

File: arm_model/urdf/arm_simple.xacro (robot description, xacro)
@@ -156,5 +156,5 @@
     <origin xyz="0 0 ${base_height/2}" rpy="0 0 0"/>
     <axis xyz="0 1 0"/>
-    <limit lower="-1.57" upper="1.57" effort="${joint_effort}" velocity="${joint_velocity}"/>
+    <limit lower="0" upper="1.57" effort="${joint_effort}" velocity="${joint_velocity}"/>
     <dynamics damping="${joint_damping}" friction="0.1"/>
   </joint>
@@ -198,5 +198,5 @@
     <origin xyz="0 0 ${first_arm_length}" rpy="0 0 0"/>
     <axis xyz="0 1 0"/>
-    <limit lower="-3.14" upper="3.14" effort="${joint_effort}" velocity="${joint_velocity}"/>
+    <limit lower="0" upper="3.14" effort="${joint_effort}" velocity="${joint_velocity}"/>
     <dynamics damping="${joint_damping}" friction="0.1"/>
   </joint>
@@ -240,5 +240,5 @@
     <origin xyz="0 0 ${second_arm_length}" rpy="0 0 0"/>
     <axis xyz="0 1 0"/>
-    <limit lower="-3.14" upper="3.14" effort="${joint_effort}" velocity="${joint_velocity}"/>
+    <limit lower="0" upper="3.14" effort="${joint_effort}" velocity="${joint_velocity}"/>
     <dynamics damping="${joint_damping}" friction="0.1"/>
   </joint>
@@ -287,3 +287,63 @@
     </plugin>
   </gazebo>
+  <!-- 障碍物：固定立方体（位于机械臂运动路径上，需避障） -->
+  <!-- <link name="obstacle">
+    <inertial>
+      <mass value="10.0"/>
+      <origin xyz="0 0 0"/>
+      <inertia ixx="1.0" ixy="0" ixz="0"
+               iyy="1.0" iyz="0"
+               izz="1.0"/>
+    </inertial>
+    <visual>
+      <origin xyz="0 0 0.05"/>
+      <geometry>
+        <box size="0.1 0.1 0.1"/>
+      </geometry>
+      <material name="black">
+        <color rgba="0 0 0 1"/>
+      </material>
+    </visual>
+    <collision>
+      <origin xyz="0 0 0.05"/>
+      <geometry>
+        <box size="0.1 0.1 0.1"/>
+      </geometry>
+    </collision>
+  </link> -->
+  <!-- 障碍物固定到世界坐标系（位置：x=0.3, y=0.1, z=0.2，在机械臂工作空间内） -->
+ <!-- <joint name="obstacle_to_world" type="fixed">
+    <parent link="world"/>
+    <child link="obstacle"/>
+    <origin xyz="0 0.2 0.3" rpy="0 0 0"/>
+  </joint> -->
+<!-- 新增：虚拟末端链接（second_arm_link 的终点） -->
+<link name="second_arm_end">
+  <!-- 无惯性（质量为0，不影响动力学） -->
+  <inertial>
+    <mass value="0.0"/>
+    <inertia ixx="0.0" ixy="0.0" ixz="0.0"
+             iyy="0.0" iyz="0.0"
+             izz="0.0"/>
+  </inertial>
+  <!-- 可视化（可选，小原点标记终点，方便观察） -->
+  <visual>
+    <geometry>
+      <sphere radius="0.005"/> <!-- 小原点，颜色为红色 -->
+    </geometry>
+    <material name="red"/>
+  </visual>
+  <!-- 无碰撞体（不影响避障） -->
+  <collision>
+    <geometry>
+      <sphere radius="0.001"/>
+    </geometry>
+  </collision>
+</link>
+<!-- 新增：固定关节，将虚拟末端链接到 second_arm_link 的终点 -->
+<joint name="second_arm_to_end" type="fixed">
+  <parent link="second_arm_link"/>
+  <child link="second_arm_end"/>
+  <origin xyz="0 0 ${second_arm_length}" rpy="0 0 0"/> <!-- 沿 Z 轴平移到 second_arm_link 的终点 -->
+</joint>
 </robot>

Commit message: avoid and link_constraint work

File: arm_model/urdf/arm_simple.xacro (robot description, xacro)
@@ -77,5 +77,5 @@
     <parent link="world"/>
     <child link="base_link"/>
-    <origin xyz="0 0 ${base_height/2}" rpy="0 0 0"/>
+    <origin xyz="3 4.495 0.68" rpy="0 0 0"/>
   </joint>
   <link name="turret_link">
@@ -316,5 +316,5 @@
     <parent link="world"/>
     <child link="obstacle"/>
-    <origin xyz="0 0.2 0.3" rpy="0 0 0"/>
+    <origin xyz="0 0.3 0.4" rpy="0 0 0"/>
   </joint> -->
 <!-- 新增：虚拟末端链接（second_arm_link 的终点） -->
@@ -347,3 +347,10 @@
   <origin xyz="0 0 ${second_arm_length}" rpy="0 0 0"/> <!-- 沿 Z 轴平移到 second_arm_link 的终点 -->
 </joint>
+  <!-- 引入场地模型（zwei.urdf） -->
+  <!-- <xacro:include filename="$(find zwei)/urdf/zwei.urdf" />
+  <joint name="arena_to_world" type="fixed">
+    <parent link="world" />
+    <child link="arena_base_link" />
+    <origin xyz="0 0 0.05" rpy="0 0 0" />
+  </joint> -->
 </robot>

File: zwei/urdf/zwei.urdf (robot description, URDF)
Before this commit: robot zwei, 36 links, 35 joints
Links:
- removed link base_link
- added link arena_base_link, mass 32830.9811175371
Joints:
- joint 25: parent base_link -> arena_base_link
- joint 26: parent base_link -> arena_base_link
- joint 27: parent base_link -> arena_base_link
- joint 28: parent base_link -> arena_base_link
- joint 29: parent base_link -> arena_base_link
- joint 30: parent base_link -> arena_base_link
- joint 31: parent base_link -> arena_base_link
- joint 32: parent base_link -> arena_base_link
- joint 33: parent base_link -> arena_base_link
- joint 34: parent base_link -> arena_base_link
- joint 35: parent base_link -> arena_base_link
- joint 36: parent base_link -> arena_base_link
- joint R1: parent base_link -> arena_base_link
- joint R2: parent base_link -> arena_base_link
- joint empytblue: parent base_link -> arena_base_link
- joint fake: parent base_link -> arena_base_link
- joint ink1: parent base_link -> arena_base_link
- joint ink10: parent base_link -> arena_base_link
- joint ink11: parent base_link -> arena_base_link
- joint ink12: parent base_link -> arena_base_link
- joint ink13: parent base_link -> arena_base_link
- joint ink14: parent base_link -> arena_base_link
- joint ink15: parent base_link -> arena_base_link
- joint ink16: parent base_link -> arena_base_link
- joint ink17: parent base_link -> arena_base_link
- joint ink18: parent base_link -> arena_base_link
- joint ink2: parent base_link -> arena_base_link
- joint ink3: parent base_link -> arena_base_link
- joint ink4: parent base_link -> arena_base_link
- joint ink5: parent base_link -> arena_base_link
- joint ink6: parent base_link -> arena_base_link
- joint ink7: parent base_link -> arena_base_link
- joint ink8: parent base_link -> arena_base_link
- joint ink9: parent base_link -> arena_base_link
- joint red: parent base_link -> arena_base_link

Commit message: add serial

File: arm_model/urdf/arm_simple.xacro (robot description, xacro)
@@ -74,8 +74,13 @@
     </collision>
   </link>
+  <!-- <joint name="world_to_base_fixed" type="fixed">
+    <parent link="world"/>
+    <child link="base_link"/>
+    <origin xyz="3 4.495 0.68" rpy="0 0 0"/>
+  </joint> -->
   <joint name="world_to_base_fixed" type="fixed">
     <parent link="world"/>
     <child link="base_link"/>
-    <origin xyz="3 4.495 0.68" rpy="0 0 0"/>
+    <origin xyz="0 0 0" rpy="0 0 0"/>
   </joint>
   <link name="turret_link">

Commit message: add arm_serial

File: arm_model/urdf/arm_simple.xacro (robot description, xacro)
@@ -6,12 +6,12 @@
   <xacro:property name="gap_between_base_turret" value="0" />
   <xacro:property name="first_arm_length" value="0.45857" />
-  <xacro:property name="first_arm_radius" value="0.03" />
+  <xacro:property name="first_arm_radius" value="0.01" />
   <xacro:property name="first_arm_mass" value="0.5" />
   <xacro:property name="second_arm_length" value="0.41476" />
-  <xacro:property name="second_arm_radius" value="0.03" />
+  <xacro:property name="second_arm_radius" value="0.01" />
   <xacro:property name="second_arm_mass" value="0.5" />
   <!-- 添加第三连杆属性 -->
   <xacro:property name="third_arm_length" value="0.1335" />
-  <xacro:property name="third_arm_radius" value="0.03" />
+  <xacro:property name="third_arm_radius" value="0.01" />
   <xacro:property name="third_arm_mass" value="0.3" />
   <!-- 添加末端小球属性 -->
